Commit message: working lidar3DFilter

File: components/hardware/laser/lidar3DFilter/robots/P3Bot/P3Bot.urdf (robot description, URDF)
Before this commit: robot P3Bot_description, 56 links, 55 joints
Links:
- removed link rotation_link
- removed link world
- link base_link: geometry collision mesh filename=robots/P3Bot/meshes/base_link.STL; visual mesh filename=robots/P3Bot/meshes/base_link.STL
- link cap: geometry collision mesh filename=robots/P3Bot/meshes/cap.STL; visual mesh filename=robots/P3Bot/meshes/cap.STL
- link chess: geometry collision mesh filename=robots/P3Bot/meshes/chess.STL; visual mesh filename=robots/P3Bot/meshes/chess.STL
- link left_arm: geometry collision mesh filename=robots/P3Bot/meshes/arm_base_link.STL; visual mesh filename=robots/P3Bot/meshes/arm_base_link.STL
- link left_arm_bracelet_link: geometry collision mesh filename=robots/P3Bot/meshes/bracelet_with_vision_link.STL; visual mesh filename=robots/P3Bot/meshes/bracelet_with_vision_link.STL
- link left_arm_forearm_link: geometry collision mesh filename=robots/P3Bot/meshes/forearm_link.STL; visual mesh filename=robots/P3Bot/meshes/forearm_link.STL
- link left_arm_half_arm_1_link: geometry collision mesh filename=robots/P3Bot/meshes/half_arm_1_link.STL; visual mesh filename=robots/P3Bot/meshes/half_arm_1_link.STL
- link left_arm_half_arm_2_link: geometry collision mesh filename=robots/P3Bot/meshes/half_arm_2_link.STL; visual mesh filename=robots/P3Bot/meshes/half_arm_2_link.STL
- link left_arm_left_inner_finger: geometry collision mesh filename=robots/P3Bot/meshes/collision/robotiq_arg2f_85_inner_finger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 scale=0.001 0.001 0.001; visual mesh filename=robots/P3Bot/meshes/visual/robotiq_arg2f_85_inner_finger.dae scale=0.001 0.001 0.001
- link left_arm_left_inner_knuckle: geometry collision mesh filename=robots/P3Bot/meshes/collision/robotiq_arg2f_85_inner_knuckl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 scale=0.001 0.001 0.001; visual mesh filename=robots/P3Bot/meshes/visual/robotiq_arg2f_85_inner_knuckle.d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 scale=0.001 0.001 0.001
- link left_arm_left_outer_finger: geometry collision mesh filename=robots/P3Bot/meshes/collision/robotiq_arg2f_85_outer_finger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 scale=0.001 0.001 0.001; visual mesh filename=robots/P3Bot/meshes/visual/robotiq_arg2f_85_outer_finger.dae scale=0.001 0.001 0.001
- link left_arm_left_outer_knuckle: geometry collision mesh filename=robots/P3Bot/meshes/collision/robotiq_arg2f_85_outer_knuckl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 scale=0.001 0.001 0.001; visual mesh filename=robots/P3Bot/meshes/visual/robotiq_arg2f_85_outer_knuckle.d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 scale=0.001 0.001 0.001
- link left_arm_right_inner_finger: geometry collision mesh filename=robots/P3Bot/meshes/collision/robotiq_arg2f_85_inner_finger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 scale=0.001 0.001 0.001; visual mesh filename=robots/P3Bot/meshes/visual/robotiq_arg2f_85_inner_finger.dae scale=0.001 0.001 0.001
- link left_arm_right_inner_knuckle: geometry collision mesh filename=robots/P3Bot/meshes/collision/robotiq_arg2f_85_inner_knuckl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 scale=0.001 0.001 0.001; visual mesh filename=robots/P3Bot/meshes/visual/robotiq_arg2f_85_inner_knuckle.d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 scale=0.001 0.001 0.001
- link left_arm_right_outer_finger: geometry collision mesh filename=robots/P3Bot/meshes/collision/robotiq_arg2f_85_outer_finger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 scale=0.001 0.001 0.001; visual mesh filename=robots/P3Bot/meshes/visual/robotiq_arg2f_85_outer_finger.dae scale=0.001 0.001 0.001
- link left_arm_right_outer_knuckle: geometry collision mesh filename=robots/P3Bot/meshes/collision/robotiq_arg2f_85_outer_knuckl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 scale=0.001 0.001 0.001; visual mesh filename=robots/P3Bot/meshes/visual/robotiq_arg2f_85_outer_knuckle.d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 scale=0.001 0.001 0.001
- link left_arm_robotiq_arg2f_base_link: geometry collision mesh filename=robots/P3Bot/meshes/collision/robotiq_arg2f_base_link_85.stl; visual mesh filename=robots/P3Bot/meshes/collision/robotiq_arg2f_base_link_85.stl
- link left_arm_shoulder_link: geometry collision mesh filename=robots/P3Bot/meshes/shoulder_link.STL; visual mesh filename=robots/P3Bot/meshes/shoulder_link.STL
- link left_arm_spherical_wrist_1_link: geometry collision mesh filename=robots/P3Bot/meshes/spherical_wrist_1_link.STL; visual mesh filename=robots/P3Bot/meshes/spherical_wrist_1_link.STL
- link left_arm_spherical_wrist_2_link: geometry collision mesh filename=robots/P3Bot/meshes/spherical_wrist_2_link.STL; visual mesh filename=robots/P3Bot/meshes/spherical_wrist_2_link.STL
- link low_body: geometry collision mesh filename=robots/P3Bot/meshes/low_body.STL; visual mesh filename=robots/P3Bot/meshes/low_body.STL
- link ricoh_theta_z1: geometry collision mesh filename=robots/P3Bot/meshes/ricoh_theta_z1.STL; visual mesh filename=robots/P3Bot/meshes/ricoh_theta_z1.STL
- link right_arm: geometry collision mesh filename=robots/P3Bot/meshes/arm_base_link.STL; visual mesh filename=robots/P3Bot/meshes/arm_base_link.STL
- link right_arm_bracelet_link: geometry collision mesh filename=robots/P3Bot/meshes/bracelet_with_vision_link.STL; visual mesh filename=robots/P3Bot/meshes/bracelet_with_vision_link.STL
- link right_arm_forearm_link: geometry collision mesh filename=robots/P3Bot/meshes/forearm_link.STL; visual mesh filename=robots/P3Bot/meshes/forearm_link.STL
- link right_arm_half_arm_1_link: geometry collision mesh filename=robots/P3Bot/meshes/half_arm_1_link.STL; visual mesh filename=robots/P3Bot/meshes/half_arm_1_link.STL
- link right_arm_half_arm_2_link: geometry collision mesh filename=robots/P3Bot/meshes/half_arm_2_link.STL; visual mesh filename=robots/P3Bot/meshes/half_arm_2_link.STL
- link right_arm_left_inner_finger: geometry collision mesh filename=robots/P3Bot/meshes/collision/robotiq_arg2f_85_inner_finger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 scale=0.001 0.001 0.001; visual mesh filename=robots/P3Bot/meshes/visual/robotiq_arg2f_85_inner_finger.dae scale=0.001 0.001 0.001
- link right_arm_left_inner_knuckle: geometry collision mesh filename=robots/P3Bot/meshes/collision/robotiq_arg2f_85_inner_knuckl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 scale=0.001 0.001 0.001; visual mesh filename=robots/P3Bot/meshes/visual/robotiq_arg2f_85_inner_knuckle.d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 scale=0.001 0.001 0.001
- link right_arm_left_outer_finger: geometry collision mesh filename=robots/P3Bot/meshes/collision/robotiq_arg2f_85_outer_finger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 scale=0.001 0.001 0.001; visual mesh filename=robots/P3Bot/meshes/visual/robotiq_arg2f_85_outer_finger.dae scale=0.001 0.001 0.001
- link right_arm_left_outer_knuckle: geometry collision mesh filename=robots/P3Bot/meshes/collision/robotiq_arg2f_85_outer_knuckl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 scale=0.001 0.001 0.001; visual mesh filename=robots/P3Bot/meshes/visual/robotiq_arg2f_85_outer_knuckle.d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 scale=0.001 0.001 0.001
- link right_arm_right_inner_finger: geometry collision mesh filename=robots/P3Bot/meshes/collision/robotiq_arg2f_85_inner_finger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 scale=0.001 0.001 0.001; visual mesh filename=robots/P3Bot/meshes/visual/robotiq_arg2f_85_inner_finger.dae scale=0.001 0.001 0.001
- link right_arm_right_inner_knuckle: geometry collision mesh filename=robots/P3Bot/meshes/collision/robotiq_arg2f_85_inner_knuckl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 scale=0.001 0.001 0.001; visual mesh filename=robots/P3Bot/meshes/visual/robotiq_arg2f_85_inner_knuckle.d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 scale=0.001 0.001 0.001
- link right_arm_right_outer_finger: geometry collision mesh filename=robots/P3Bot/meshes/collision/robotiq_arg2f_85_outer_finger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 scale=0.001 0.001 0.001; visual mesh filename=robots/P3Bot/meshes/visual/robotiq_arg2f_85_outer_finger.dae scale=0.001 0.001 0.001
- link right_arm_right_outer_knuckle: geometry collision mesh filename=robots/P3Bot/meshes/collision/robotiq_arg2f_85_outer_knuckl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 scale=0.001 0.001 0.001; visual mesh filename=robots/P3Bot/meshes/visual/robotiq_arg2f_85_outer_knuckle.d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 scale=0.001 0.001 0.001
- link right_arm_robotiq_arg2f_base_link: geometry collision mesh filename=robots/P3Bot/meshes/collision/robotiq_arg2f_base_link_85.stl; visual mesh filename=robots/P3Bot/meshes/collision/robotiq_arg2f_base_link_85.stl
- link right_arm_shoulder_link: geometry collision mesh filename=robots/P3Bot/meshes/shoulder_link.STL; visual mesh filename=robots/P3Bot/meshes/shoulder_link.STL
- link right_arm_spherical_wrist_1_link: geometry collision mesh filename=robots/P3Bot/meshes/spherical_wrist_1_link.STL; visual mesh filename=robots/P3Bot/meshes/spherical_wrist_1_link.STL
- link right_arm_spherical_wrist_2_link: geometry collision mesh filename=robots/P3Bot/meshes/spherical_wrist_2_link.STL; visual mesh filename=robots/P3Bot/meshes/spherical_wrist_2_link.STL
- link rs_helios: geometry collision mesh filename=robots/P3Bot/meshes/rs_helios.STL; visual mesh filename=robots/P3Bot/meshes/rs_helios.STL
Joints:
- removed joint base_rotation_joint
- removed joint base_translation_joint

Commit message: lidar3DFilter work

File: components/hardware/laser/lidar3DFilter/robots/P3Bot/P3Bot.urdf (robot description, URDF)
Before this commit: robot robots/P3Bot, 54 links, 53 joints
Joints:
- joint base_link2low_body: origin xyz=0 0 0.21 rpy=0 0 -1.57 -> xyz=0 0.1 0.30 rpy=0 0 0
